File: hardware/pico-poe-mains-carrier/pico-poe-mains-carrier.kicad_pcb (KiCad board)
At the start: 2 copper layers, 80 x 51.5 mm, 22 parts, among them J1 230VAC L/N, U1 W5500-EVB-Pico-PoE, U2 LTV-814S, U3 SN74LVC1G14DBVR, U4 TMP1075DR

Commit message: Hardware: carrier board v1.1 - fuse, factory reset button, holes, logo
- F1 T100mA 250VAC (Schurter UMT 250, 3403.0156.11, no LCSC part) after
  the L terminal; the divider is R1 in L and R2-R4 in N, one series loop
  through F1
- SW1 (XKB TS-1187A, LCSC C318884) from GP22 to GND next to H1, so the
  firmware's 10 s factory reset works on the carrier
- I2C pull-ups renumbered R8/R9 (no gap after R7)
- H4/H5 M3 holes under the module for mounting the carrier when the
  module is on headers (project footprint without courtyard)
- Silkscreen: RF logo (logo/, flattened by generate.py), "RF-UPS-Monitor
  v1.1", "Made by Kenneth Foli Jørgensen 2026"; title blocks updated
- render.sh: male headers under the module (module 11 mm up on
  headers); refuses to run without the KiCad 3D model library
- ERC/DRC clean; fab files, renders, STEP/GLB regenerated
- README, carrier README, TODO, CHANGELOG

Co-Authored-By: Claude Opus 5.5 (1M context) <noreply@anthropic.com>
Parts:
- removed R10: 4.7k, Resistor_SMD:R_0603_1608Metric
- added F1: T100mA 250VAC, Fuse:Fuse_Schurter_UMT250, F.Cu at (103.3, 75.0)
- added H4: MountingHole_3.2mm_M3, PicoPoE_Carrier:MountingHole_3.2mm_M3_UnderModule, F.Cu at (70.0, 50.5)
- added H5: MountingHole_3.2mm_M3, PicoPoE_Carrier:MountingHole_3.2mm_M3_UnderModule, F.Cu at (106.5, 50.5)
- added R8: 4.7k, Resistor_SMD:R_0603_1608Metric, F.Cu at (57.6, 80.2)
- added SW1: FACTORY RESET, Button_Switch_SMD:SW_Push_1P1T_XKB_TS-1187A, F.Cu at (51.5, 64.9)
- moved R2 12.7 mm to (106.6, 69.9)
- moved R1 8.00 mm to (95.0, 75.0)
- moved R9 4.75 mm to (53.0, 79.0), turned to 90 degrees
- moved R3 2.10 mm to (100.9, 69.9)
Connections:
- net /N_MID renamed /N_MID2
- R1 pad 1: /L_MID -> /OPTO_A
- R1 pad 2: /AC_L -> /L_FUSED
- R2 pad 1: /OPTO_A -> /N_MID1
- R2 pad 2: /L_MID -> /AC_N
- R3 pad 2: /AC_N -> /N_MID1
- R9 pad 1: /I2C_SDA -> /I2C_SCL
- U1 pad 29: unconnected-(U1-GP22-Pad29) -> /FACTORY_RESET
Routing:
- net /FACTORY_RESET: track 0.00 -> 41.6 mm
- net /L_MID: track 5.07 -> 0.00 mm
- net /AC_N: track 10.3 -> 6.74 mm
- net /AC_L: track 10.3 -> 7.25 mm
- net /N_MID1: track 0.00 -> 2.78 mm
- net /L_FUSED: track 0.00 -> 2.59 mm
- net /N_MID2: track 5.07 -> 2.97 mm
Other:
- board text added: "Made by Kenneth Foli Jørgensen 2026"
- board text added: "RESET 10s"
- board text added: "RF-UPS-Monitor v1.1"
- board text removed: "Pico-PoE Mains Monitor v1.0"
