File: hardware/pico-poe-mains-carrier/pico-poe-mains-carrier.kicad_sch (KiCad schematic)
At the start: 22 parts, among them J1 230VAC L/N, U1 W5500-EVB-Pico-PoE, U2 LTV-814S, U3 SN74LVC1G14DBVR, U4 TMP1075DR

Commit message: Hardware: carrier board v1.1 - fuse, factory reset button, holes, logo
- F1 T100mA 250VAC (Schurter UMT 250, 3403.0156.11, no LCSC part) after
  the L terminal; the divider is R1 in L and R2-R4 in N, one series loop
  through F1
- SW1 (XKB TS-1187A, LCSC C318884) from GP22 to GND next to H1, so the
  firmware's 10 s factory reset works on the carrier
- I2C pull-ups renumbered R8/R9 (no gap after R7)
- H4/H5 M3 holes under the module for mounting the carrier when the
  module is on headers (project footprint without courtyard)
- Silkscreen: RF logo (logo/, flattened by generate.py), "RF-UPS-Monitor
  v1.1", "Made by Kenneth Foli Jørgensen 2026"; title blocks updated
- render.sh: male headers under the module (module 11 mm up on
  headers); refuses to run without the KiCad 3D model library
- ERC/DRC clean; fab files, renders, STEP/GLB regenerated
- README, carrier README, TODO, CHANGELOG

Co-Authored-By: Claude Opus 5.5 (1M context) <noreply@anthropic.com>
Parts:
- removed R10: 4.7k, Resistor_SMD:R_0603_1608Metric, symbol PicoPoE_Carrier:R
- added F1: T100mA 250VAC, Fuse:Fuse_Schurter_UMT250, symbol PicoPoE_Carrier:Fuse
- added H4, H5: MountingHole_3.2mm_M3, PicoPoE_Carrier:MountingHole_3.2mm_M3_UnderModule, symbol PicoPoE_Carrier:MountingHole
- added R8: 4.7k, Resistor_SMD:R_0603_1608Metric, symbol PicoPoE_Carrier:R
- added SW1: FACTORY RESET, Button_Switch_SMD:SW_Push_1P1T_XKB_TS-1187A, symbol PicoPoE_Carrier:SW_Push
Connections:
- net +3V3: now also R8.2
- net AC_L: now also F1.2; no longer R1.2
- net AC_N: now also R2.2; no longer R3.2
- net GND: now also SW1.2
- net I2C_SCL: now also R9.1
- net I2C_SDA: now also R8.1; no longer R9.1
- net OPTO_A: now also R1.1; no longer R2.1
- net FACTORY_RESET: now reaches U1.29 (GP22)
- net FACTORY_RESET: now also SW1.1
- removed net L_MID: R1.1, R2.2
- net N_MID renamed N_MID2
- new net L_FUSED: F1.1, R1.2
- new net N_MID1: R2.1, R3.2
- no-connect marks 30 -> 29
Other:
- note added: "F1 T100mA 250VAC in the only current loop. 4x 68k 1206 (>=200V): ~1.2 mA peak, ~50 mW each. LTV-814S AC-input optocoupler, 5 kVrms. PCB: >=6.5 mm clearance, >=6.4 mm creepage + routed slot."
- note added: "GP16..GP21 are used by the on-board W5500 - do not use. GP27 (pin 32) = MAINS_OK input: HIGH = 230VAC present. GP4/GP5 = I2C0 SDA/SCL to TMP1075 (address 0x48). GP22 (pin 29) = SW1 to GND: hold 10 s for a factory reset (internal pull-up). +3V3 comes from the module's 3V3(OUT) pin 36 (PoE powered)."
- note removed: "4x 68k 1206 (>=200V) split between L and N: ~1.2 mA peak, ~50 mW each. LTV-814S AC-input optocoupler, 5 kVrms. PCB: >=7.5 mm creepage + routed slot."
- note removed: "GP16..GP21 are used by the on-board W5500 - do not use. GP27 (pin 32) = MAINS_OK input: HIGH = 230VAC present. GP4/GP5 = I2C0 SDA/SCL to TMP1075 (address 0x48). +3V3 comes from the module's 3V3(OUT) pin 36 (PoE powered)."
- company: (none) -> Kenneth Foli Jørgensen
- title: W5500-EVB-Pico-PoE mains monitor carrier -> RF-UPS-Monitor carrier for the W5500-EVB-Pico-PoE
